File: DB1NV_Antennenverstärker.kicad_pcb (KiCad board)
At the start: 2 copper layers, 39.5 x 20 mm, 36 parts, among them P1 CONN_01X01_Antenne, P2 CONN_01X02, Q1 BF 545A, Q2 BF 199, Q3 BF 324, U1 LM7812ACT

Commit message: gefertigte Version...
Parts:
- removed L2: 100µH, lpis2812:L-PIS2812
- removed U1: LM7812ACT, Housings_SOIC:SOIC-8_3.9x4.9mm_Pitch1.27mm
- added C14: 4,7µ X7R, Capacitors_SMD:C_0805, F.Cu at (142.6, 98.5)
- added IC1: LT3042, Housings_DFN_QFN:DFN-10-1EP_3x3mm_Pitch0.5mm, F.Cu at (147.4, 96.9)
- added R14: 8,5k, Resistors_SMD:R_0603, F.Cu at (151.0, 96.4)
- added R15: 1,2k, Resistors_SMD:R_0603, F.Cu at (151.2, 94.0)
- added R16: 121k, Resistors_SMD:R_0603, F.Cu at (142.8, 94.5)
- added R17: 69k, Resistors_SMD:R_0603, F.Cu at (145.7, 94.0)
- added R18: 1.8k, Resistors_SMD:R_0603, F.Cu at (148.5, 94.0)
- C12: value 100n -> 4.7u; footprint Capacitors_SMD:C_0603 -> Capacitors_SMD:C_0805
- moved C5 6.60 mm to (149.4, 100.8)
- moved C11 6.09 mm to (153.3, 99.1), turned to 270 degrees
- moved C10 3.89 mm to (151.0, 99.3), turned to 270 degrees
- moved C12 3.49 mm to (142.6, 96.4)
- moved C13 3.15 mm to (145.1, 103.0), turned to 180 degrees
- moved C4 0.30 mm to (144.4, 100.8), turned to 180 degrees
Routing:
- net GND: track 57.9 -> 78.4 mm, vias 16 -> 44
- net Net-(C12-Pad1): track 18.8 -> 4.24 mm
- net Net-(IC1-Pad3): track 0.00 -> 5.06 mm
- net Net-(IC1-Pad6): track 0.00 -> 3.35 mm
- net Net-(C10-Pad1): track 11.0 -> 13.7 mm
- net VAA: track 29.7 -> 29.2 mm, vias 0 -> 2
- added copper zone on F.Cu, net Net-(C10-Pad1)
- added copper zone on F.Cu, net Net-(C3-Pad1)
- added copper zone on F.Cu, net Net-(C9-Pad1)
- added copper zone on F.Cu, net VAA
Other:
- outline, holes or cut-outs redrawn
- board text added: "PHörauf 2015"
