File: DB1NV_Antennenverstärker.sch (KiCad schematic (older format))
At the start: 41 parts, among them IC1 LT3042, P1 CONN_01X01_Antenne, P2 CONN_01X02, Q1 BF 545A, Q2 BF 199, Q3 BF 324

Commit message: gefertigte Version...
Parts:
- C12: footprint (none) -> Capacitors_SMD:C_0805
- IC1: footprint (none) -> Housings_DFN_QFN:DFN-10-1EP_3x3mm_Pitch0.5mm
- R14, R15, R16, R17, R18: footprint (none) -> Resistors_SMD:R_0603
Connections:
- net GND: now also IC1.11 (Pad)
Changed lines of the file:
@@
 	0    1    1    0
 $EndComp
-Wire Wire Line
-	9200 1900 10350 1900
 Connection ~ 9300 1900
 $Comp
@@
 	1    0    0    -1
 $EndComp
-Connection ~ 10350 1900
 $Comp
 L LT3042 IC1
@@
 F 0 "IC1" H 8450 1650 60  0000 C CNN
 F 1 "LT3042" H 8600 2250 60  0000 C CNN
-F 2 "" H 8950 1950 60  0001 C CNN
+F 2 "Housings_DFN_QFN:DFN-10-1EP_3x3mm_Pitch0.5mm" H 8950 1950 60  0001 C CNN
 F 3 "" H 8950 1950 60  0000 C CNN
 	1    8700 1950
@@
 F 0 "R16" V 8730 2600 50  0000 C CNN
 F 1 "121k" V 8650 2600 50  0000 C CNN
-F 2 "" V 8580 2600 30  0001 C CNN
+F 2 "Resistors_SMD:R_0603" V 8580 2600 30  0001 C CNN
 F 3 "" H 8650 2600 30  0000 C CNN
 	1    8650 2600
@@
 F 0 "C12" H 8475 2700 50  0000 L CNN
 F 1 "4.7u" H 8475 2500 50  0000 L CNN
-F 2 "" H 8488 2450 30  0001 C CNN
+F 2 "Capacitors_SMD:C_0805" H 8488 2450 30  0001 C CNN
 F 3 "" H 8450 2600 60  0000 C CNN
 	1    8450 2600
@@
 F 0 "R17" V 9380 2050 50  0000 C CNN
 F 1 "69k" V 9300 2050 50  0000 C CNN
-F 2 "" V 9230 2050 30  0001 C CNN
+F 2 "Resistors_SMD:R_0603" V 9230 2050 30  0001 C CNN
 F 3 "" H 9300 2050 30  0000 C CNN
 	1    9300 2050
@@
 F 0 "R18" V 9380 2350 50  0000 C CNN
 F 1 "1.8k" V 9300 2350 50  0000 C CNN
-F 2 "" V 9230 2350 30  0001 C CNN
+F 2 "Resistors_SMD:R_0603" V 9230 2350 30  0001 C CNN
 F 3 "" H 9300 2350 30  0000 C CNN
 	1    9300 2350
@@
 F 0 "R15" V 8030 2250 50  0000 C CNN
 F 1 "1,2k" V 7950 2250 50  0000 C CNN
-F 2 "" V 7880 2250 30  0001 C CNN
+F 2 "Resistors_SMD:R_0603" V 7880 2250 30  0001 C CNN
 F 3 "" H 7950 2250 30  0000 C CNN
 	1    7950 2250
@@
 F 0 "R14" V 8030 1950 50  0000 C CNN
 F 1 "8,5k" V 7950 1950 50  0000 C CNN
-F 2 "" V 7880 1950 30  0001 C CNN
+F 2 "Resistors_SMD:R_0603" V 7880 1950 30  0001 C CNN
 F 3 "" H 7950 1950 30  0000 C CNN
 	1    7950 1950
@@
 Wire Wire Line
 	8050 2000 8200 2000
-Connection ~ 7750 2750
 NoConn ~ 8200 2100
 Text Notes 8250 1150 0    60   ~ 0
@@
 	1    0    0    -1
 $EndComp
+Wire Wire Line
+	9900 1900 9200 1900
+$Comp
+L GND #PWR?
+U 1 1 558EBB81
+P 8700 1500
+F 0 "#PWR?" H 8700 1250 50  0001 C CNN
+F 1 "GND" H 8700 1350 50  0000 C CNN
+F 2 "" H 8700 1500 60  0000 C CNN
+F 3 "" H 8700 1500 60  0000 C CNN
+	1    8700 1500
+	-1   0    0    1
+$EndComp
 $EndSCHEMATC
